Commit message: add mecanum wheel meshes

File: bme_gazebo_basics/urdf/mogi_bot_mecanum.urdf (robot description, URDF)
Before this commit: robot mogi_bot, 6 links, 5 joints
Links:
- link base_link: geometry collision box size=.4 .2 .1; visual mesh filename=package://bme_gazebo_basics/meshes/mogi_bot.dae
- link front_left_wheel: geometry collision sphere radius=.1; visual mesh filename=package://bme_gazebo_basics/meshes/mecanum_wheel_left.STL scale=0.002 .002 0.002
- link front_right_wheel: geometry collision sphere radius=.1; visual mesh filename=package://bme_gazebo_basics/meshes/mecanum_wheel_right.STL scale=0.002 .002 0.002
- link rear_left_wheel: geometry collision sphere radius=.1; visual mesh filename=package://bme_gazebo_basics/meshes/mecanum_wheel_right.STL scale=0.002 .002 0.002
- link rear_right_wheel: geometry collision sphere radius=.1; visual mesh filename=package://bme_gazebo_basics/meshes/mecanum_wheel_left.STL scale=0.002 .002 0.002
