Commit message: mogi bot URDF with final 3D models

File: bme_gazebo_basics/urdf/mogi_bot.urdf (robot description, URDF)
Before this commit: robot mogi_bot, 4 links, 3 joints
Links:
- link base_link: geometry collision box size=.4 .2 .1; collision sphere radius=0.0499
- link left_wheel: geometry collision cylinder length=.05 radius=.1; visual mesh filename=package://bme_gazebo_basics/meshes/wheel.dae
- link right_wheel: geometry collision cylinder length=.05 radius=.1; visual mesh filename=package://bme_gazebo_basics/meshes/wheel.dae
